File: power-supply/kicad/psu.kicad_pcb (KiCad board)
At the start: 2 copper layers, 23 x 22.1 mm, 14 parts, among them J3 SSQ-103-03-G-D, U1 LM2776, U3 TPS72301DBVR, U5 TPS79333DBVR

Commit message: Update KiCad designs for all 3 boards and re-export gerbers
- bias-control-lt8362: schematic + PCB updates, exported gerbers
  including new B_Paste/F_Paste layers
- power-supply: schematic + PCB updates, re-exported gerbers with new
  naming (.gbl/.gbs/.gto/.gtl/.gts) replacing old .gbr files, added
  paste layer exports
- tiav3_s14160: schematic + PCB updates, re-exported gerbers with new
  naming, added paste layer exports
- fp-lib-table updates across all four board projects
- new "w paste" gerber zip exports for assembly
Parts:
- added J1: Snibbor Inc LOGO, snibbor_logos:snibbor_inc_logo, F.Cu at (205.1, 105.8)
- added J2: Bennet LOGO, snibbor_logos:Bennett logo close 1 layered, B.Cu at (204.3, 106.6)
- added J4: Bennet full LOGO, snibbor_logos:Bennett logo full 1 layered, B.Cu at (193.3, 94.4)
Connections:
- J3 pad 4: (no net) -> unconnected-(J3-Pin_4-Pad4)
- J3 pad 5: (no net) -> /BIAS
