File: power-supply/kicad/psu.kicad_sch (KiCad schematic)
At the start: 14 parts, among them J3 SSQ-103-03-G-D, U1 LM2776, U3 TPS72301DBVR, U5 TPS79333DBVR

Commit message: Update KiCad designs for all 3 boards and re-export gerbers
- bias-control-lt8362: schematic + PCB updates, exported gerbers
  including new B_Paste/F_Paste layers
- power-supply: schematic + PCB updates, re-exported gerbers with new
  naming (.gbl/.gbs/.gto/.gtl/.gts) replacing old .gbr files, added
  paste layer exports
- tiav3_s14160: schematic + PCB updates, re-exported gerbers with new
  naming, added paste layer exports
- fp-lib-table updates across all four board projects
- new "w paste" gerber zip exports for assembly
Parts:
- added J1: Snibbor Inc LOGO, snibbor_logos:snibbor_inc_logo, symbol Logo:Conn_NC
- added J2: Bennett LOGO, snibbor_logos:Bennett logo close 1 layered, symbol Logo:Conn_NC
- added J4: Bennett full LOGO, snibbor_logos:Bennett logo full 1 layered, symbol Logo:Conn_NC
