File: bias-control-lt8362/bias_generator_LT8362.kicad_pcb (KiCad board)
At the start: 4 copper layers, 37.6 x 30.6 mm, 61 parts, among them IC1 LT8361EMSE/LT8362EMSE, IC2 ATSAMD21E18A-AF, IC4 MCP47FEB22A2-E_ST, J1 ISP, J2 Conn_01x04, J3 Conn_01x06, J4 USB_C_Receptacle_USB2.0_16P, U1 MIC5317-3.3YM5-TR, U2 RT9072B, U3 MCP6C02T-020E/CHY

Commit message: Update KiCad designs for all 3 boards and re-export gerbers
- bias-control-lt8362: schematic + PCB updates, exported gerbers
  including new B_Paste/F_Paste layers
- power-supply: schematic + PCB updates, re-exported gerbers with new
  naming (.gbl/.gbs/.gto/.gtl/.gts) replacing old .gbr files, added
  paste layer exports
- tiav3_s14160: schematic + PCB updates, re-exported gerbers with new
  naming, added paste layer exports
- fp-lib-table updates across all four board projects
- new "w paste" gerber zip exports for assembly
Parts:
- added J5: Snibbor Inc LOGO, snibbor_logos:snibbor_inc_logo, F.Cu at (193.1, 116.3)
- added J6: Bennett LOGO, snibbor_logos:Bennett logo close 1 layered, B.Cu at (178.0, 103.6)
- added J7: Bennett full LOGO, snibbor_logos:Bennett logo full 1 layered, F.Cu at (178.4, 91.9)

Commit message: sourcing, ordering, and assembling
Parts:
- U2: value RT9072B -> RT9072B(ob)/LT3014ES5#TRP
Changed lines of the file:
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@@
 			)
 		)
+		(property ki_fp_filters "Connector*:*")
+		(sheetname "/")
+		(sheetfile "bias_generator_LT8362.kicad_sch")
 		(attr exclude_from_pos_files)
 		(fp_poly
@@
 			)
 		)
-		(property "Value" "RT9072B"
+		(property "Value" "RT9072B(ob)/LT3014ES5#TRP"
 			(at 0 2.9 0)
 			(layer "F.Fab")
@@
 			)
 		)
+		(property ki_fp_filters "Connector*:*")
+		(sheetname "/")
+		(sheetfile "bias_generator_LT8362.kicad_sch")
 		(attr smd)
 		(fp_poly
@@
 			)
 		)
+		(property ki_fp_filters "Connector*:*")
+		(sheetname "/")
+		(sheetfile "bias_generator_LT8362.kicad_sch")
 		(attr smd)
 		(fp_poly
